Commit message: 3

File: src/diff_drive_robot/description/robot.urdf.xacro (robot description, xacro)
@@ -3,3 +3,6 @@
     <!-- include xacro files-->
     <xacro:include filename="robot_core.xacro"/>
+    <xacro:include filename="gazebo_control.xacro"/>
+    <xacro:include filename="lidar.xacro"/>
+    <xacro:include filename="camera.xacro"/>
 </robot>

File: src/diff_drive_robot/description/robot_core.xacro (robot description, xacro)
@@ -15,4 +15,7 @@
     <material name="black">
         <color rgba="0 0 0 1"/>
+    </material>
+    <material name="red">
+        <color rgba="1 0 0 1"/>
     </material>
     <!-- base link -->
@@ -43,4 +46,9 @@
         </xacro:inertial_box>
     </link>
+    <gazebo reference ="chassis">
+        <material>
+            Gazebo/White
+        </material>
+    </gazebo>
     <!-- left wheel joint and link -->
     <joint name="left_wheel_joint" type="continuous">
@@ -67,4 +75,9 @@
         </xacro:inertial_cylinder>
     </link>
+    <gazebo reference ="left_wheel">
+        <material>
+            Gazebo/Orange
+        </material>
+    </gazebo>
     <!-- left wheel joint and link -->
     <joint name="right_wheel_joint" type="continuous">
@@ -91,4 +104,9 @@
         </xacro:inertial_cylinder>
     </link>
+    <gazebo reference ="right_wheel">
+        <material>
+            Gazebo/Orange
+        </material>
+    </gazebo>
     <!-- caster wheel joint and link -->
     <joint name="caster_wheel_joint" type="fixed">
@@ -100,5 +118,5 @@
         <visual>
             <geometry>
-                <sphere radius="0.4"/>
+                <sphere radius="0.04"/>
             </geometry>
             <material name="blue"/>
@@ -106,10 +124,17 @@
         <collision>
             <geometry>
-                <sphere radius="0.4"/>
+                <sphere radius="0.04"/>
             </geometry>
         </collision>
+        <xacro:inertial_sphere mass="0.1" radius="0.04">
+            <origin xyz="0.0 0.0 0.0" rpy="0.0 0.0 0.0"/>
+        </xacro:inertial_sphere>
     </link>
-    <xacro:inertial_sphere mass="0.1" radius="0.04">
-        <origin xyz="0.0 0.0 0.0" rpy="0.0 0.0 0.0"/>
-    </xacro:inertial_sphere>
+    <gazebo reference ="caster_wheel">
+        <material>
+            Gazebo/Blue
+        </material>
+        <mu1 value = "0.001" />
+        <mu2 value = "0.001" />
+    </gazebo>
 </robot>

Commit message: 4

File: src/diff_drive_robot/description/robot.urdf.xacro (robot description, xacro)
@@ -3,5 +3,6 @@
     <!-- include xacro files-->
     <xacro:include filename="robot_core.xacro"/>
-    <xacro:include filename="gazebo_control.xacro"/>
+    <!-- <xacro:include filename="gazebo_control.xacro"/> -->
+    <xacro:include filename="ros2_control.xacro"/>
     <xacro:include filename="lidar.xacro"/>
     <xacro:include filename="camera.xacro"/>

File: src/diff_drive_robot/description/robot_core.xacro (robot description, xacro)
@@ -21,4 +21,12 @@
     <!-- base link -->
     <link name="base_link">
+    </link>
+    <!-- Base Footprint -->
+    <joint name="base_footprint_joint" type="fixed">
+        <parent link="base_link"/>
+        <child link="base_footprint"/>
+        <origin xyz="0.0 0.0 0.0" rpy="0.0 0.0 0.0"/>
+    </joint>
+    <link name="base_footprint">
     </link>
     <!-- chassis joint and link -->
